Commit message: grasp test

File: fmauch_universal_robot/final_test/config/gazebo_hrc_sim.urdf (robot description, URDF)
Before this commit: robot hrc_sim, 39 links, 38 joints
Joints:
- joint azure_kinect_fix_1: origin xyz=0.5 0 1 rpy=0 1.5707963267948966 0 -> xyz=-0.5 0 1 rpy=1.5707963267948966 1.5707963267948966 0
- joint world_to_world_camera_joint: origin xyz=0.0 0.0 1.0 rpy=0 0 0 -> xyz=0.0 0.0 1.0 rpy=0 0 3.1416

Commit message: path

File: fmauch_universal_robot/final_test/config/gazebo_hrc_sim.urdf (robot description, URDF)
Before this commit: robot hrc_sim, 39 links, 38 joints
Joints:
- joint azure_kinect_fix_1: origin xyz=-0.5 0 1 rpy=1.5707963267948966 1.5707963267948966 0 -> xyz=-0.5 0 1 rpy=0 1.5707963267948966 3.141592653589793

Commit message: code update

File: fmauch_universal_robot/final_test/config/gazebo_hrc_sim.urdf (robot description, URDF)
Before this commit: robot hrc_sim, 39 links, 38 joints
Joints:
- joint azure_kinect_fix_1: origin xyz=-0.5 0 1 rpy=0 1.5707963267948966 3.141592653589793 -> xyz=-0.5 0 1 rpy=0 1.5707963267948966 -3.141592653589793
