Commit message: master

File: Azure_Kinect_ROS_Driver/urdf/azure_kinect_1.urdf.xacro (robot description, xacro)
@@ -11,5 +11,5 @@
             <origin xyz="0 0 0" rpy="0 0 0"/>
             <geometry>
-                <box size="0.001 0.001 0.001" />
+                <box size="0.00001 0.00001 0.00001" />
             </geometry>
             <material name="grey">

File: fmauch_universal_robot/ur_gazebo/urdf/hrc_sim.xacro (robot description, xacro)
@@ -49,5 +49,5 @@
     <xacro:include filename="$(find azure_kinect_ros_driver)/urdf/azure_kinect_1.urdf.xacro" />
     <xacro:azure_kinect_1 prefix="${prefix}" parent="${prefix}world_camera" >
-        <origin xyz="0.5 0 1" rpy="0 ${pi/2} 0"/>
+        <origin xyz="0.5 0 1" rpy="${pi} ${pi/2} 0"/>
     </xacro:azure_kinect_1>
         <!-- Define camera_base_optical as a child, not a root link -->
@@ -63,7 +63,6 @@
         <material>Gazebo/Black</material>
         <sensor name="camera_1" type="depth">
-            <pose> 0 0 0 0 0 0 </pose>
-            <visualize>true</visualize>
-            <update_rate>10</update_rate>
+            <always_on>true</always_on>
+            <update_rate>20.0</update_rate>
             <camera>
                 <horizontal_fov>1.089</horizontal_fov>
@@ -78,9 +77,21 @@
                 </clip>
             </camera>
-            <plugin name="camera_controller_1" filename="libgazebo_ros_camera.so">
-                <frame_name>camera_base_optical_1</frame_name>
-                <cameraName>azure_kinect_camera_1</cameraName>
-                <min_depth>0.1</min_depth>
-                <max_depth>10</max_depth>
+            <plugin name="camera_controller_1" filename="libgazebo_ros_openni_kinect.so">
+                <baseline>0.1</baseline>
+		        <alwaysOn>true</alwaysOn>
+		        <updateRate>10</updateRate>
+		        <cameraName>azure_kinect_camera_1</cameraName>
+		        <imageTopicName>depth/image_raw</imageTopicName>
+		        <cameraInfoTopicName>depth/camera_info</cameraInfoTopicName>
+		        <depthImageTopicName>depth/image_raw</depthImageTopicName>
+		        <depthImageCameraInfoTopicName>depth/camera_info</depthImageCameraInfoTopicName>
+		        <pointCloudTopicName>depth/points</pointCloudTopicName>
+		        <frameName>camera_base_optical_1</frameName>
+		        <pointCloudCutoff>0.3</pointCloudCutoff>
+		        <distortion_k1>0.0</distortion_k1>
+		        <distortion_k2>0.0</distortion_k2>
+		        <distortion_k3>0.0</distortion_k3>
+		        <distortion_t1>0.0</distortion_t1>
+		        <distortion_t2>0.0</distortion_t2>
             </plugin>
         </sensor>
@@ -101,5 +112,5 @@
     <gazebo reference="camera_base">
         <material>Gazebo/Black</material>
-        <sensor name="camera" type="depth">
+        <sensor type="depth" name="camera">
             <pose> 0 0 0 0 0 0 </pose>
             <visualize>true</visualize>
@@ -117,9 +128,21 @@
                 </clip>
             </camera>
-            <plugin name="camera_controller" filename="libgazebo_ros_camera.so">
-                <frame_name>camera_base_optical</frame_name>
-                <cameraName>azure_kinect_camera</cameraName>
-                <min_depth>0.1</min_depth>
-                <max_depth>10</max_depth>
+            <plugin name="camera_controller" filename="libgazebo_ros_openni_kinect.so">
+                <baseline>0.1</baseline>
+		        <alwaysOn>true</alwaysOn>
+		        <updateRate>10</updateRate>
+		        <cameraName>azure_kinect_camera</cameraName>
+		        <imageTopicName>depth/image_raw</imageTopicName>
+		        <cameraInfoTopicName>depth/camera_info</cameraInfoTopicName>
+		        <depthImageTopicName>depth/image_raw</depthImageTopicName>
+		        <depthImageCameraInfoTopicName>depth/camera_info</depthImageCameraInfoTopicName>
+		        <pointCloudTopicName>depth/points</pointCloudTopicName>
+		        <frameName>camera_base_optical</frameName>
+		        <pointCloudCutoff>0.3</pointCloudCutoff>
+		        <distortion_k1>0.0</distortion_k1>
+		        <distortion_k2>0.0</distortion_k2>
+		        <distortion_k3>0.0</distortion_k3>
+		        <distortion_t1>0.0</distortion_t1>
+		        <distortion_t2>0.0</distortion_t2>
             </plugin>
         </sensor>

File: robotiq_85_gripper/robotiq_85_description/urdf/robotiq_85_gripper.urdf.xacro (robot description, xacro)
@@ -303,14 +303,13 @@
             <arm>
               <arm_name>gripper_arm</arm_name>
-              <palm_link>${prefix}gripper_finger1_inner_knuckle_link</palm_link>
+              <palm_link>${parent}</palm_link>
               <gripper_link>${prefix}gripper_finger1_finger_tip_link</gripper_link>
-              <palm_link>${prefix}gripper_finger2_inner_knuckle_link</palm_link>
               <gripper_link>${prefix}gripper_finger2_finger_tip_link</gripper_link>
             </arm>
 	    <forces_angle_tolerance>100</forces_angle_tolerance>
-	    <update_rate>20</update_rate>
+	    <update_rate>2</update_rate>
 	    <grip_count_threshold>1</grip_count_threshold>
-	    <max_grip_count>3</max_grip_count>
-	    <release_tolerance>0.0198</release_tolerance>
+	    <max_grip_count>2</max_grip_count>
+	    <release_tolerance>0.005</release_tolerance>
 	    <disable_collisions_on_attach>true</disable_collisions_on_attach>
 	    <contact_topic>__default_topic__</contact_topic>
